File: muxbreakout.sch (KiCad schematic (older format))
At the start: 3 parts, among them J1 1x10_pins_L, J2 1x10_pins_R, U1 mux

Commit message: fixed pitch
Parts:
- J1, J2: footprint (none) -> muxbreakout:pins
- U1: footprint (none) -> muxbreakout:muxbreakout
Changed lines of the file:
@@
 F 0 "U1" H 5700 2400 60  0000 C CNN
 F 1 "mux" H 5700 3400 60  0000 C CNN
-F 2 "" H 5350 2800 60  0001 C CNN
+F 2 "muxbreakout:muxbreakout" H 5350 2800 60  0001 C CNN
 F 3 "" H 5350 2800 60  0001 C CNN
 	1    5700 3250
@@
 F 0 "J2" H 7450 3100 50  0000 L CNN
 F 1 "1x10_pins_R" H 7300 3200 50  0000 L CNN
-F 2 "" H 6950 3350 50  0001 C CNN
+F 2 "muxbreakout:pins" H 6950 3350 50  0001 C CNN
 F 3 "" H 6950 3350 50  0001 C CNN
 	1    6950 3200
@@
 F 0 "J1" H 3900 3100 50  0000 C CNN
 F 1 "1x10_pins_L" H 3900 3200 50  0000 C CNN
-F 2 "" H 4450 3200 50  0001 C CNN
+F 2 "muxbreakout:pins" H 4450 3200 50  0001 C CNN
 F 3 "" H 4450 3200 50  0001 C CNN
 	1    4450 3200
